File: PTL-RAIL/PTL-RAIL.kicad_sch (KiCad schematic)
At the start: 0 parts

Commit message: PTL-RAIL: LED row on top edge, TSOP row on bottom edge, node parts aligned at 84 mm pitch; J3/J4 10-way and J5/J6 4-way screw terminals
Other:
- sheet CAN ports: added {CAN}; removed none
- sheet ESP32 ports: added {CAN}, {RX_NODE}, {TX_NODE}; removed none
- sheet Power ports: added +3V3, +5V; removed none
- sheet RX nodes ports: added {RX_NODE}; removed none
- sheet TX nodes ports: added {TX_NODE}; removed none
- note removed: "PTL-RAIL rev A - top level. Same PCB fits top, middle and bottom rail positions by population."

Commit message: PTL-RAIL: IR shrouds, bottom-side node parts, test points, SW4 user button
- 3D-printed shroud outlines (28 mm) with M3 mounting holes on every LED
  and TSOP node, replicated from node 2; parts cleared from shroud areas
- TX/RX node resistors, caps and MOSFETs moved to the bottom layer and
  arranged uniformly per node
- Filleted the TSOP output bus corners; solid zone connection on the
  starved-thermal GND pads
- Silkscreen cleanup: uniform 0.8 mm refs, connector pin labels on both
  sides, J5/J6 mirrored labels, node TX/RX labels, title/company/date
- Redundant GND vias and a GND via fence along the board edge
- Mid-board mounting holes (H25-H28) and 4 mm rounded corners concentric
  with the corner holes
- Test points TP5-TP19 (TX_1-5, TSOP_OUT_1-5, VIN, +5V, +3V3, 2x GND)
  in schematic and PCB, routed
- SW4 generic user push button with R34 10k pull-up
Other:
- sheet ESP32 ports: added {TSOP_OUT}; removed {RX_NODE}
- sheet RX nodes ports: added {TSOP_OUT}; removed {RX_NODE}
Changed lines of the file:
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@@
 			)
 		)
-		(pin "{RX_NODE}" bidirectional
-			(at 177.8 139.7 0)
+		(pin "{TX_NODE}" bidirectional
+			(at 177.8 101.6 0)
 			(effects
 				(font
@@
 			)
 		)
-		(pin "{TX_NODE}" bidirectional
-			(at 177.8 101.6 0)
+		(pin "{TSOP_OUT}" bidirectional
+			(at 177.8 139.7 0)
 			(effects
 				(font
@@
 			)
 		)
-		(pin "{RX_NODE}" bidirectional
+		(pin "{TSOP_OUT}" bidirectional
 			(at 190.5 139.7 180)
 			(effects
