File: PTL-RAIL/PTL-RAIL.kicad_pcb (KiCad board)
At the start: 2 copper layers, 440 x 60 mm, 4 parts

Commit message: PTL-RAIL: LED row on top edge, TSOP row on bottom edge, node parts aligned at 84 mm pitch; J3/J4 10-way and J5/J6 4-way screw terminals
Parts:
- added C1: 2.2uF, Capacitor_SMD:C_1210_3225Metric, F.Cu at (728.7, 670.0)
- added C10: 0.1uF, Capacitor_SMD:C_0805_2012Metric, F.Cu at (616.3, 665.6)
- added C11: 1uF, Capacitor_SMD:C_0805_2012Metric, F.Cu at (626.5, 670.1)
- added C12: 10uF, Capacitor_SMD:C_0805_2012Metric, F.Cu at (621.2, 664.8)
- added C13: 10uF, Capacitor_SMD:C_0805_2012Metric, F.Cu at (623.2, 664.8)
- added C14: 22uF, Capacitor_SMD:C_0805_2012Metric, F.Cu at (625.3, 664.8)
- added C15: 1uF, Capacitor_SMD:C_0805_2012Metric, F.Cu at (627.3, 664.8)
- added C16: 0.1uF, Capacitor_SMD:C_0805_2012Metric, F.Cu at (629.3, 664.8)
- added C17: 0.1uF, Capacitor_SMD:C_0805_2012Metric, F.Cu at (621.8, 671.3)
- added C18: 0.1uF, Capacitor_SMD:C_0805_2012Metric, F.Cu at (577.0, 668.2)
- added C19: 0.1uF, Capacitor_SMD:C_0805_2012Metric, F.Cu at (584.1, 668.2)
- added C2: 10uF, Capacitor_SMD:C_0805_2012Metric, F.Cu at (855.9, 721.0)
- added C20: 0.1uF, Capacitor_SMD:C_0805_2012Metric, F.Cu at (590.7, 667.9)
- added C21: 0.1uF, Capacitor_SMD:C_0805_2012Metric, F.Cu at (790.1, 733.4)
- added C22: 4.7 µF, Capacitor_SMD:C_0805_2012Metric, F.Cu at (422.1, 731.8)
- added C23: 4.7 µF, Capacitor_SMD:C_0805_2012Metric, F.Cu at (506.1, 731.8)
- added C24: 4.7 µF, Capacitor_SMD:C_0805_2012Metric, F.Cu at (590.1, 731.8)
- added C25: 4.7 µF, Capacitor_SMD:C_0805_2012Metric, F.Cu at (674.1, 731.8)
- added C26: 4.7 µF, Capacitor_SMD:C_0805_2012Metric, F.Cu at (758.1, 731.8)
- added C3: 2.2uF, Capacitor_SMD:C_1210_3225Metric, F.Cu at (725.4, 670.0)
- added C4: 10uF, Capacitor_SMD:C_0805_2012Metric, F.Cu at (853.6, 721.0)
- added C5: 100nF, Capacitor_SMD:C_0805_2012Metric, F.Cu at (721.5, 672.7)
- added C6: 22nF, Capacitor_SMD:C_0805_2012Metric, F.Cu at (710.9, 667.7)
- added C7: 100pF, Capacitor_SMD:C_0805_2012Metric, F.Cu at (713.2, 667.7)
- added C8: 22uF, Capacitor_SMD:C_1210_3225Metric, F.Cu at (714.0, 680.3)
- added C9: 22uF, Capacitor_SMD:C_1210_3225Metric, F.Cu at (718.2, 680.3)
- added CR1: PESD1CAN_215, Package_TO_SOT_SMD:SOT-23, F.Cu at (801.3, 728.2)
- added D1: SS36, Diode_SMD:D_SMC, F.Cu at (714.9, 674.5)
- added D10: IR333C, LED_THT:LED_D5.0mm_Horizontal_O1.27mm_Z3.0mm_IRGrey, F.Cu at (669.9, 658.0)
- added D11: IR333C, LED_THT:LED_D5.0mm_Horizontal_O1.27mm_Z3.0mm_IRGrey, F.Cu at (753.9, 658.0)
- added D2: LED, LED_SMD:LED_0805_2012Metric, F.Cu at (755.0, 769.5)
- added D3: SS14, Diode_SMD:D_SMA, F.Cu at (616.3, 671.6)
- added D4: WS2812B, LED_SMD:LED_WS2812B_PLCC4_5.0x5.0mm_P3.2mm, F.Cu at (578.0, 673.0)
- added D5: WS2812B, LED_SMD:LED_WS2812B_PLCC4_5.0x5.0mm_P3.2mm, F.Cu at (584.6, 673.0)
- added D6: WS2812B, LED_SMD:LED_WS2812B_PLCC4_5.0x5.0mm_P3.2mm, F.Cu at (591.3, 673.0)
- added D7: IR333C, LED_THT:LED_D5.0mm_Horizontal_O1.27mm_Z3.0mm_IRGrey, F.Cu at (417.9, 658.0)
- added D8: IR333C, LED_THT:LED_D5.0mm_Horizontal_O1.27mm_Z3.0mm_IRGrey, F.Cu at (501.9, 658.0)
- added D9: IR333C, LED_THT:LED_D5.0mm_Horizontal_O1.27mm_Z3.0mm_IRGrey, F.Cu at (585.9, 658.0)
- added J1: JST_PH_4P, Connector_JST:JST_PH_B4B-PH-K_1x04_P2.00mm_Vertical, F.Cu at (614.8, 682.8)
- added J3: Screw_Terminal_01x10, TerminalBlock_4Ucon:TerminalBlock_4Ucon_1x10_P3.50mm_Horizontal, F.Cu at (401.8, 676.6)
- added J4: Screw_Terminal_01x10, TerminalBlock_4Ucon:TerminalBlock_4Ucon_1x10_P3.50mm_Horizontal, F.Cu at (433.3, 668.7)
- added J5: Screw_Terminal_01x04, TerminalBlock_4Ucon:TerminalBlock_4Ucon_1x04_P3.50mm_Horizontal, F.Cu at (394.7, 666.2)
- added J6: Screw_Terminal_01x04, TerminalBlock_4Ucon:TerminalBlock_4Ucon_1x04_P3.50mm_Horizontal, F.Cu at (738.1, 678.2)
- added L1: 15uH, Inductor_SMD:L_APV_ANR8040, F.Cu at (705.3, 675.5)
- added Q1: AO3400A, Package_TO_SOT_SMD:SOT-23, F.Cu at (416.6, 639.7)
- added Q2: AO3400A, Package_TO_SOT_SMD:SOT-23, F.Cu at (500.6, 639.8)
- added Q3: AO3400A, Package_TO_SOT_SMD:SOT-23, F.Cu at (586.5, 639.4)
- added Q4: AO3400A, Package_TO_SOT_SMD:SOT-23, F.Cu at (666.7, 632.2)
- added Q5: AO3400A, Package_TO_SOT_SMD:SOT-23, F.Cu at (764.8, 638.4)
- added R1: 274k, Resistor_SMD:R_0805_2012Metric, F.Cu at (724.3, 664.7)
- added R10: 100k, Resistor_SMD:R_0805_2012Metric, F.Cu at (412.1, 637.7)
- added R11: 180R, Resistor_SMD:R_0805_2012Metric, F.Cu at (421.1, 638.7)
- added R12: 100R, Resistor_SMD:R_0805_2012Metric, F.Cu at (496.1, 640.8)
- added R13: 100k, Resistor_SMD:R_0805_2012Metric, F.Cu at (496.1, 637.8)
- added R14: 180R, Resistor_SMD:R_0805_2012Metric, F.Cu at (505.1, 638.8)
- added R15: 100R, Resistor_SMD:R_0805_2012Metric, F.Cu at (582.0, 640.4)
- added R16: 100k, Resistor_SMD:R_0805_2012Metric, F.Cu at (582.0, 637.4)
- added R17: 180R, Resistor_SMD:R_0805_2012Metric, F.Cu at (591.0, 638.4)
- added R18: 100R, Resistor_SMD:R_0805_2012Metric, F.Cu at (662.2, 633.2)
- added R19: 100k, Resistor_SMD:R_0805_2012Metric, F.Cu at (662.2, 630.2)
- added R2: 8.45k, Resistor_SMD:R_0805_2012Metric, F.Cu at (712.4, 664.6)
- added R20: 180R, Resistor_SMD:R_0805_2012Metric, F.Cu at (671.2, 631.2)
- added R21: 100R, Resistor_SMD:R_0805_2012Metric, F.Cu at (760.3, 639.4)
- added R22: 100k, Resistor_SMD:R_0805_2012Metric, F.Cu at (760.3, 636.4)
- added R23: 180R, Resistor_SMD:R_0805_2012Metric, F.Cu at (769.3, 637.4)
- added R24: 100R, Resistor_SMD:R_0805_2012Metric, F.Cu at (414.1, 731.8)
- added R25: 100R, Resistor_SMD:R_0805_2012Metric, F.Cu at (419.2, 731.8)
- added R26: 100R, Resistor_SMD:R_0805_2012Metric, F.Cu at (498.1, 731.8)
- added R27: 100R, Resistor_SMD:R_0805_2012Metric, F.Cu at (503.2, 731.8)
- added R28: 100R, Resistor_SMD:R_0805_2012Metric, F.Cu at (582.1, 731.8)
- added R29: 100R, Resistor_SMD:R_0805_2012Metric, F.Cu at (587.2, 731.8)
- added R3: 60.4k, Resistor_SMD:R_0805_2012Metric, F.Cu at (706.6, 667.7)
- added R30: 100R, Resistor_SMD:R_0805_2012Metric, F.Cu at (666.1, 731.8)
- added R31: 100R, Resistor_SMD:R_0805_2012Metric, F.Cu at (671.2, 731.8)
- added R32: 100R, Resistor_SMD:R_0805_2012Metric, F.Cu at (750.1, 731.8)
- added R33: 100R, Resistor_SMD:R_0805_2012Metric, F.Cu at (755.2, 731.8)
- added R4: 11.5k, Resistor_SMD:R_0805_2012Metric, F.Cu at (708.6, 667.7)
- added R5: 1k, Resistor_SMD:R_0805_2012Metric, F.Cu at (751.5, 769.5)
- added R6: 10k, Resistor_SMD:R_0805_2012Metric, F.Cu at (626.5, 668.1)
- added R7: 120R, Resistor_SMD:R_0805_2012Metric, F.Cu at (801.3, 733.7)
- added R8: 10k, Resistor_SMD:R_0805_2012Metric, F.Cu at (801.3, 731.7)
- added R9: 100R, Resistor_SMD:R_0805_2012Metric, F.Cu at (412.1, 640.7)
- added REF**: JST_EH_B10B-EH-A_1x10_P2.50mm_Vertical, Connector_JST:JST_EH_B10B-EH-A_1x10_P2.50mm_Vertical, F.Cu at (338.3, 686.0)
- added SW1: SW_SPST, Button_Switch_SMD:SW_SPST_PTS645Sx43SMTR92, F.Cu at (705.8, 776.6)
- added SW2: SW_SPST, Button_Switch_SMD:SW_SPST_PTS645Sx43SMTR92, F.Cu at (705.8, 784.5)
- added SW3: SW_DIP_x01, Button_Switch_THT:SW_DIP_SPSTx01_Slide_9.78x4.72mm_W7.62mm_P2.54mm, F.Cu at (798.0, 727.6)
- added TP1: USBC_D+, TestPoint:TestPoint_Pad_D1.5mm, F.Cu at (619.2, 684.8)
- added TP2: USBC_D-, TestPoint:TestPoint_Pad_D1.5mm, F.Cu at (619.2, 674.8)
- added TP3: USB_D+, TestPoint:TestPoint_Pad_D1.5mm, F.Cu at (623.6, 682.8)
- added TP4: USB_D-, TestPoint:TestPoint_Pad_D1.5mm, F.Cu at (623.6, 676.8)
- added U1: TLV1117-33, Package_TO_SOT_SMD:SOT-223-3_TabPin2, F.Cu at (853.6, 714.1)
- added U10: TSOP382xx, OptoDevice:Vishay_MINICAST-3Pin, F.Cu at (750.1, 688.0)
- added U2: TPS54360BQDDARQ1, 0_IC:TPS54360BQDDARQ1, F.Cu at (718.8, 667.9)
- added U3: ESP32-S3-WROOM-1, RF_Module:ESP32-S3-WROOM-1U, F.Cu at (640.6, 673.0)
- added U4: USBLC6-2SC6, Package_TO_SOT_SMD:SOT-23-6, F.Cu at (620.3, 679.8)
- added U5: SN65HVD230DR, Package_SO:SOIC-8_3.9x4.9mm_P1.27mm, F.Cu at (795.1, 733.3)
- added U6: TSOP382xx, OptoDevice:Vishay_MINICAST-3Pin, F.Cu at (414.1, 688.0)
- added U7: TSOP382xx, OptoDevice:Vishay_MINICAST-3Pin, F.Cu at (498.1, 688.0)
- added U8: TSOP382xx, OptoDevice:Vishay_MINICAST-3Pin, F.Cu at (582.1, 688.0)
- added U9: TSOP382xx, OptoDevice:Vishay_MINICAST-3Pin, F.Cu at (666.1, 688.0)
- moved H1 704.7 mm to (388.6, 647.0)
- moved H3 704.7 mm to (388.6, 699.0)
- moved H2 684.8 mm to (780.6, 647.0)
- moved H4 684.8 mm to (780.6, 699.0)
Other:
- board size 440 x 60 mm -> 400 x 43.8 mm
- board text added: "BOTTOM EDGE: TSOP row, lens down, reading the bin below; outputs to J3 OUT -> board below ESP32 IO4-8"
- board text added: "TOP EDGE: IR LED row (IR333C horizontal), firing up into the bin above; gates from this board ESP32 IO9-13"
- board text removed: "FRONT 32-60 mm: node band, solid GND pour both faces, shroud keep-outs"
- board text removed: "FRONT EDGE (throw side)"
- board text removed: "N5"
- board text removed: "Nodes at 84 mm pitch, first at x=52 (42 mm from the 420 mm opening edge). LED at node-6, TSOP at node+6, y=49.5 from rear edge"
- board text removed: "REAR 0-32 mm: electronics, connectors, ESP32 (antenna at rear edge)"
- board text removed: "REAR EDGE"
- board text removed: "RX"
- board text removed: "TX"

Commit message: PTL-RAIL: place TX/RX node MOSFETs, resistors and caps next to their LED/TSOP
Parts:
- moved C2 164.1 mm to (697.5, 678.2)
- moved C4 164.1 mm to (695.2, 678.2)
- moved U1 164.1 mm to (695.1, 671.4)
- moved R24 44.4 mm to (411.7, 687.5)
- moved R25 44.4 mm to (421.5, 687.5)
- moved R26 44.4 mm to (495.7, 687.5)
- moved R27 44.4 mm to (505.5, 687.5)
- moved R28 44.4 mm to (579.7, 687.5)
- moved R29 44.4 mm to (589.5, 687.5)
- moved R30 44.4 mm to (663.7, 687.5)
- moved R31 44.4 mm to (673.5, 687.5)
- moved R32 44.4 mm to (747.7, 687.5)
- moved R33 44.4 mm to (757.5, 687.5)
- moved C22 44.3 mm to (423.6, 687.5)
- moved C23 44.3 mm to (507.6, 687.5)
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Other:
- board size 400 x 43.8 mm -> 400 x 40 mm

Commit message: PTL-RAIL: TSOP Vs decoupling caps on the Vs node; place CAN, buttons, status LED and mounting holes
Parts:
- moved R7 367.6 mm to (440.0, 666.0)
- moved CR1 367.0 mm to (438.5, 673.0), turned to 0 degrees
- moved R8 363.4 mm to (441.5, 680.5), turned to 0 degrees
- moved SW3 359.8 mm to (443.5, 666.0), turned to 0 degrees
- moved U5 352.8 mm to (447.0, 676.5), turned to 180 degrees
- moved C21 342.0 mm to (453.0, 676.0), turned to 270 degrees
- moved D2 186.1 mm to (600.3, 666.0)
- moved R5 181.6 mm to (600.3, 669.0)
- moved SW1 159.1 mm to (600.3, 657.5)
- moved SW2 145.0 mm to (600.3, 685.0)
- moved H1 10.0 mm to (388.6, 657.0)
- moved H2 10.0 mm to (780.6, 657.0)
- moved H3 10.0 mm to (388.6, 689.0)
- moved H4 10.0 mm to (780.6, 689.0)
- moved C22 2.10 mm to (421.5, 687.5), turned to 270 degrees
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Connections:
- C22 pad 2: +3V3 -> Net-(U6-Vs)
- C23 pad 2: +3V3 -> Net-(U7-Vs)
- C24 pad 2: +3V3 -> Net-(U8-Vs)
- C25 pad 2: +3V3 -> Net-(U9-Vs)
- C26 pad 2: +3V3 -> Net-(U10-Vs)

Commit message: PTL-RAIL: move CAN block (U5, C21, CR1, R7, R8, SW3) to mid-board, flip node Q1-Q5/C22-C26 rotation, relocate SW1/SW2, shift C24/R28/R29
PCB only, no tracks yet:
- CAN transceiver U5 with C21, CR1, R7, R8 and SW3 moved from x~440 to x~550-565.
- Q1-Q5 and C22-C26 rotation 270 -> -90; C24, R28, R29 moved down to y 698.1.
- SW1 moved to x 618.9; SW2 moved to (649.4, 678.1) rotated 90.
- Two unreferenced M3 mounting holes (REF**) added at (576.8, 688.2) and (592.5, 688.2); one gr_rect added.
Parts:
- added REF**: MountingHole_3.2mm_M3, MountingHole:MountingHole_3.2mm_M3, F.Cu at (592.5, 688.2)
- added REF**: MountingHole_3.2mm_M3, MountingHole:MountingHole_3.2mm_M3, F.Cu at (576.8, 688.2)
- moved CR1 126.8 mm to (565.3, 671.4), turned to 180 degrees
- moved R7 124.4 mm to (563.8, 678.4), turned to 180 degrees
- moved R8 121.9 mm to (562.3, 663.9), turned to 180 degrees
- moved SW3 117.4 mm to (560.3, 678.4), turned to 180 degrees
- moved U5 110.1 mm to (556.8, 667.9), turned to 0 degrees
- moved C21 98.1 mm to (550.8, 668.4), turned to 90 degrees
- moved SW2 49.6 mm to (649.4, 678.1), turned to 90 degrees
- moved SW1 18.6 mm to (618.9, 657.5)
- moved C24 10.6 mm to (589.5, 698.1)
- moved R28 10.6 mm to (579.7, 698.1)
- moved R29 10.6 mm to (591.6, 698.1)

Commit message: PTL-RAIL: IR shrouds, bottom-side node parts, test points, SW4 user button
- 3D-printed shroud outlines (28 mm) with M3 mounting holes on every LED
  and TSOP node, replicated from node 2; parts cleared from shroud areas
- TX/RX node resistors, caps and MOSFETs moved to the bottom layer and
  arranged uniformly per node
- Filleted the TSOP output bus corners; solid zone connection on the
  starved-thermal GND pads
- Silkscreen cleanup: uniform 0.8 mm refs, connector pin labels on both
  sides, J5/J6 mirrored labels, node TX/RX labels, title/company/date
- Redundant GND vias and a GND via fence along the board edge
- Mid-board mounting holes (H25-H28) and 4 mm rounded corners concentric
  with the corner holes
- Test points TP5-TP19 (TX_1-5, TSOP_OUT_1-5, VIN, +5V, +3V3, 2x GND)
  in schematic and PCB, routed
- SW4 generic user push button with R34 10k pull-up
Parts:
- removed REF**: JST_EH_B10B-EH-A_1x10_P2.50mm_Vertical, Connector_JST:JST_EH_B10B-EH-A_1x10_P2.50mm_Vertical
- added G***: LOGO, LOGO, F.Cu at (612.3, 676.8)
- added G***: LOGO, LOGO, B.Cu at (611.2, 676.7)
- added H11: MountingHole_3.2mm_M3, MountingHole:MountingHole_3.2mm_M3, F.Cu at (658.6, 688.0)
- added H12: MountingHole_3.2mm_M3, MountingHole:MountingHole_3.2mm_M3, F.Cu at (678.6, 688.0)
- added H13: MountingHole_3.2mm_M3, MountingHole:MountingHole_3.2mm_M3, F.Cu at (742.6, 688.0)
- added H14: MountingHole_3.2mm_M3, MountingHole:MountingHole_3.2mm_M3, F.Cu at (762.6, 688.0)
- added H15: MountingHole_3.2mm_M3, MountingHole:MountingHole_3.2mm_M3, F.Cu at (406.6, 658.0)
- added H16: MountingHole_3.2mm_M3, MountingHole:MountingHole_3.2mm_M3, F.Cu at (426.6, 658.0)
- added H17: MountingHole_3.2mm_M3, MountingHole:MountingHole_3.2mm_M3, F.Cu at (490.6, 658.0)
- added H18: MountingHole_3.2mm_M3, MountingHole:MountingHole_3.2mm_M3, F.Cu at (510.6, 658.0)
- added H19: MountingHole_3.2mm_M3, MountingHole:MountingHole_3.2mm_M3, F.Cu at (574.6, 658.0)
- added H20: MountingHole_3.2mm_M3, MountingHole:MountingHole_3.2mm_M3, F.Cu at (594.6, 658.0)
- added H21: MountingHole_3.2mm_M3, MountingHole:MountingHole_3.2mm_M3, F.Cu at (658.6, 658.0)
- added H22: MountingHole_3.2mm_M3, MountingHole:MountingHole_3.2mm_M3, F.Cu at (678.6, 658.0)
- added H23: MountingHole_3.2mm_M3, MountingHole:MountingHole_3.2mm_M3, F.Cu at (742.6, 658.0)
- added H24: MountingHole_3.2mm_M3, MountingHole:MountingHole_3.2mm_M3, F.Cu at (762.6, 658.0)
- added H25: MountingHole_M3, MountingHole:MountingHole_3.2mm_M3_Pad, F.Cu at (479.2, 686.2)
- added H26: MountingHole_M3, MountingHole:MountingHole_3.2mm_M3_Pad, F.Cu at (606.0, 658.6)
- added H27: MountingHole_M3, MountingHole:MountingHole_3.2mm_M3_Pad, F.Cu at (688.8, 658.6)
- added H28: MountingHole_M3, MountingHole:MountingHole_3.2mm_M3_Pad, F.Cu at (630.1, 687.7)
- added H5: MountingHole_3.2mm_M3, MountingHole:MountingHole_3.2mm_M3, F.Cu at (406.6, 688.0)
- added H6: MountingHole_3.2mm_M3, MountingHole:MountingHole_3.2mm_M3, F.Cu at (426.6, 688.0)
- added H7: MountingHole_3.2mm_M3, MountingHole:MountingHole_3.2mm_M3, F.Cu at (490.6, 688.0)
- added H8: MountingHole_3.2mm_M3, MountingHole:MountingHole_3.2mm_M3, F.Cu at (510.6, 688.0)
- added R34: 10k, Resistor_SMD:R_0805_2012Metric, F.Cu at (628.1, 674.0)
- added SW4: SW_SPST, Button_Switch_SMD:SW_SPST_PTS645Sx43SMTR92, F.Cu at (634.4, 673.0)
- added TP10: TSOP_OUT_1, TestPoint:TestPoint_Loop_D1.80mm_Drill1.0mm_Beaded, F.Cu at (414.1, 680.8)
- added TP11: TSOP_OUT_2, TestPoint:TestPoint_Loop_D1.80mm_Drill1.0mm_Beaded, F.Cu at (482.5, 667.5)
- added TP12: TSOP_OUT_3, TestPoint:TestPoint_Loop_D1.80mm_Drill1.0mm_Beaded, F.Cu at (581.9, 680.8)
- added TP13: TSOP_OUT_4, TestPoint:TestPoint_Loop_D1.80mm_Drill1.0mm_Beaded, F.Cu at (666.1, 680.8)
- added TP14: TSOP_OUT_5, TestPoint:TestPoint_Loop_D1.80mm_Drill1.0mm_Beaded, F.Cu at (750.1, 680.8)
- added TP15: VIN, TestPoint:TestPoint_Loop_D1.80mm_Drill1.0mm_Beaded, F.Cu at (721.5, 658.3)
- added TP16: +5V, TestPoint:TestPoint_Loop_D1.80mm_Drill1.0mm_Beaded, F.Cu at (710.5, 682.3)
- added TP17: +3V3, TestPoint:TestPoint_Loop_D1.80mm_Drill1.0mm_Beaded, F.Cu at (689.6, 674.5)
- added TP18: GND, TestPoint:TestPoint_Loop_D1.80mm_Drill1.0mm_Beaded, F.Cu at (705.0, 685.5)
- added TP19: GND, TestPoint:TestPoint_Loop_D1.80mm_Drill1.0mm_Beaded, F.Cu at (626.0, 684.0)
- added TP5: TX_1, TestPoint:TestPoint_Loop_D1.80mm_Drill1.0mm_Beaded, F.Cu at (440.0, 669.1)
- added TP6: TX_2, TestPoint:TestPoint_Loop_D1.80mm_Drill1.0mm_Beaded, F.Cu at (516.5, 683.2)
- added TP7: TX_3, TestPoint:TestPoint_Loop_D1.80mm_Drill1.0mm_Beaded, F.Cu at (550.0, 682.9)
- added TP8: TX_4, TestPoint:TestPoint_Loop_D1.80mm_Drill1.0mm_Beaded, F.Cu at (669.1, 672.4)
- added TP9: TX_5, TestPoint:TestPoint_Loop_D1.80mm_Drill1.0mm_Beaded, F.Cu at (753.0, 672.8)
- C22, C23, C24, C25, C26, Q1, Q2, Q3, Q4, Q5, R10, R11, R12, R13, R14, R15, R16, R17, R18, R19, R20, R21, R22, R23, R24, R25, R26, R27, R28, R29, R30, R31, R32, R33, R9: moved to B.Cu
- U3: footprint RF_Module:ESP32-S3-WROOM-1U -> RF_Module:ESP32-S3-WROOM-1
- moved R5 101.3 mm to (701.5, 664.4)
- moved D2 97.4 mm to (697.7, 664.4)
- moved SW1 96.8 mm to (522.2, 661.1), turned to 180 degrees
- moved SW2 90.9 mm to (558.7, 684.9)
- moved C17 89.9 mm to (526.6, 680.3), turned to 90 degrees
- moved TP4 85.9 mm to (532.0, 678.5), turned to 0 degrees
- moved D3 84.9 mm to (526.8, 685.8), turned to -90 degrees
- moved TP2 83.9 mm to (530.0, 682.8), turned to 0 degrees
- moved C11 83.5 mm to (537.4, 666.8)
- moved C13 83.5 mm to (534.1, 661.5)
- moved C16 83.5 mm to (540.2, 661.5)
- moved R6 83.5 mm to (537.4, 664.8)
- moved C12 83.5 mm to (532.1, 661.5)
- moved C14 83.5 mm to (536.1, 661.5)
- moved C15 83.5 mm to (538.2, 661.5)
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- renumbered REF** to H10, REF** to H9
Connections:
- CR1 pad 1: CAN_L -> CAN_H
- CR1 pad 2: CAN_H -> CAN_L
- J4 pad 1: /ESP32/TSOP_OUT_1_ESP -> GND
- J4 pad 10: GND -> /ESP32/TSOP_OUT_1_ESP
- J4 pad 2: /ESP32/TSOP_OUT_2_ESP -> GND
- J4 pad 3: /ESP32/TSOP_OUT_3_ESP -> VIN
- J4 pad 4: /ESP32/TSOP_OUT_4_ESP -> CAN_L
- J4 pad 5: /ESP32/TSOP_OUT_5_ESP -> CAN_H
- J4 pad 6: CAN_H -> /ESP32/TSOP_OUT_5_ESP
- J4 pad 7: CAN_L -> /ESP32/TSOP_OUT_4_ESP
- J4 pad 8: VIN -> /ESP32/TSOP_OUT_3_ESP
- J4 pad 9: GND -> /ESP32/TSOP_OUT_2_ESP
- J6 pad 1: CAN_H -> GND
- J6 pad 2: CAN_L -> VIN
- J6 pad 3: VIN -> CAN_L
- J6 pad 4: GND -> CAN_H
- R24 pad 2: /RX nodes/TSOP_OUT_1 -> /ESP32/TSOP_OUT_1
- R26 pad 2: /RX nodes/TSOP_OUT_2 -> /ESP32/TSOP_OUT_2
- R28 pad 2: /RX nodes/TSOP_OUT_3 -> /ESP32/TSOP_OUT_3
- R30 pad 2: /RX nodes/TSOP_OUT_4 -> /ESP32/TSOP_OUT_4
- R32 pad 2: /RX nodes/TSOP_OUT_5 -> /ESP32/TSOP_OUT_5
- U3 pad 12: /ESP32/TSOP_OUT_1_ESP -> /ESP32/TSOP_OUT_5_ESP
- U3 pad 26: unconnected-(U3-IO45-Pad26) -> Net-(SW4-A)
Routing:
- net VIN: track 0.00 -> 479.0 mm
- net +5V: track 0.00 -> 471.2 mm, vias 0 -> 5
- net +3V3: track 0.00 -> 446.3 mm, vias 0 -> 4
- net CAN_L: track 0.00 -> 445.8 mm, vias 0 -> 5
- net CAN_H: track 0.00 -> 419.1 mm, vias 0 -> 4
- net /ESP32/TSOP_OUT_5: track 0.00 -> 329.8 mm, vias 0 -> 3
- net /ESP32/TSOP_OUT_4: track 0.00 -> 245.7 mm, vias 0 -> 3
- net /ESP32/TX_5: track 0.00 -> 214.8 mm, vias 0 -> 1
- net /ESP32/TSOP_OUT_3: track 0.00 -> 165.7 mm, vias 0 -> 3
- net /ESP32/TX_1: track 0.00 -> 159.9 mm, vias 0 -> 6
- net GND: track 0.00 -> 157.4 mm, vias 0 -> 515
- net /ESP32/TSOP_OUT_1_ESP: track 0.00 -> 137.8 mm, vias 0 -> 2
- net /ESP32/TX_4: track 0.00 -> 132.1 mm, vias 0 -> 2
- net /ESP32/TSOP_OUT_2_ESP: track 0.00 -> 132.0 mm, vias 0 -> 2
- net /ESP32/TSOP_OUT_3_ESP: track 0.00 -> 126.1 mm, vias 0 -> 2
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- added copper zone on B.Cu, net GND
- added copper zone on F.Cu, net GND
Other:
- outline, holes or cut-outs redrawn
- board text added: "3V3"
- board text added: "5V"
- board text added: "BOOT"
- board text added: "CAN / POWER"
- board text added: "CAN TERM"
- board text added: "CANH"
- board text added: "CANL"
- board text added: "D+"
- board text added: "D-"
- board text added: "GND"
- board text added: "IR TX ROW (TOP EDGE) / TSOP RX ROW (BOTTOM EDGE)"
- board text added: "PWR"
- board text added: "RST"
- board text added: "RX1"
- board text added: "RX2"
- board text added: "RX3"
- board text added: "RX4"
- board text added: "RX5"
- board text added: "STATUS"
- board text added: "TSOP IN"
- board text added: "TSOP OUT"
- board text added: "TX1"
- board text added: "TX2"
- board text added: "TX3"
- board text added: "TX4"
- board text added: "TX5"
- board text added: "USB"
- board text added: "VIN"

Commit message: PTL-RAIL: move SW4 user button to IO14 (ACK_BUTTON), add C27 100nF debounce
Parts:
- added C27: 0.1uF, Capacitor_SMD:C_0805_2012Metric, F.Cu at (553.7, 682.8)
Connections:
- R34 pad 2: Net-(SW4-A) -> /ESP32/ACK_BUTTON
- SW4 pad 1: Net-(SW4-A) -> /ESP32/ACK_BUTTON
- U3 pad 22: unconnected-(U3-IO14-Pad22) -> /ESP32/ACK_BUTTON
- U3 pad 26: Net-(SW4-A) -> unconnected-(U3-IO45-Pad26)
Routing:
- net /ESP32/ACK_BUTTON: track 0.00 -> 94.5 mm, vias 0 -> 2
- net Net-(SW4-A): track 85.5 -> 0.00 mm, vias 2 -> 0

Commit message: PTL-RAIL rev A: normalize cap values, IO45 no-connect, README and docs
- Capacitor values unified: 0.1uF -> 100nF (C10, C16-C21, C27; now one
  BOM line with C5), '4.7 µF' -> 4.7uF (C22-C26)
- No-connect flag on U3 IO45 (ERC clean apart from 2 CAN label warnings)
- Zones refilled
- PTL-RAIL/README.md: board summary, pinouts, ESP32 pin map, test points,
  mounting, fab/assembly notes, production file list, rev A open issues
- Root README points to PTL-RAIL and the release assets
Parts:
- C10, C16, C17, C18, C19, C20, C21, C27: value 0.1uF -> 100nF
- C22, C23, C24, C25, C26: value 4.7 µF -> 4.7uF
Routing:
- net +3V3: track 446.3 -> 447.3 mm
- net VIN: track 479.0 -> 480.0 mm
- net GND: vias 515 -> 624
Other:
- outline, holes or cut-outs redrawn
- board text removed: "BOTTOM EDGE: TSOP row, lens down, reading the bin below; outputs to J3 OUT -> board below ESP32 IO4-8"
- board text removed: "TOP EDGE: IR LED row (IR333C horizontal), firing up into the bin above; gates from this board ESP32 IO9-13"
