File: PTL-RAIL/esp32.kicad_sch (KiCad schematic)
At the start: 0 parts

Commit message: PTL-RAIL: LED row on top edge, TSOP row on bottom edge, node parts aligned at 84 mm pitch; J3/J4 10-way and J5/J6 4-way screw terminals
Parts:
- added C10, C16, C17, C18, C19, C20: 0.1uF, Capacitor_SMD:C_0805_2012Metric, symbol Device:C
- added C11, C15: 1uF, Capacitor_SMD:C_0805_2012Metric, symbol Device:C
- added C12, C13: 10uF, Capacitor_SMD:C_0805_2012Metric, symbol Device:C
- added C14: 22uF, Capacitor_SMD:C_0805_2012Metric, symbol Device:C
- added D3: SS14, Diode_SMD:D_SMA, symbol Diode:SS14
- added D4, D5, D6: WS2812B, LED_SMD:LED_WS2812B_PLCC4_5.0x5.0mm_P3.2mm, symbol LED:WS2812B
- added J1: JST_PH_4P, Connector_JST:JST_PH_B4B-PH-K_1x04_P2.00mm_Vertical, symbol Connector_Generic:Conn_01x04
- added J3, J4: Screw_Terminal_01x10, TerminalBlock_4Ucon:TerminalBlock_4Ucon_1x10_P3.50mm_Horizontal, symbol Connector:Screw_Terminal_01x10
- added J5, J6: Screw_Terminal_01x04, TerminalBlock_4Ucon:TerminalBlock_4Ucon_1x04_P3.50mm_Horizontal, symbol Connector:Screw_Terminal_01x04
- added R6: 10k, Resistor_SMD:R_0805_2012Metric, symbol Device:R
- added SW1, SW2: SW_SPST, Button_Switch_SMD:SW_SPST_PTS645Sx43SMTR92, symbol Switch:SW_SPST
- added TP1: USBC_D+, TestPoint:TestPoint_Pad_D1.5mm, symbol Connector:TestPoint
- added TP2: USBC_D-, TestPoint:TestPoint_Pad_D1.5mm, symbol Connector:TestPoint
- added TP3: USB_D+, TestPoint:TestPoint_Pad_D1.5mm, symbol Connector:TestPoint
- added TP4: USB_D-, TestPoint:TestPoint_Pad_D1.5mm, symbol Connector:TestPoint
- added U3: ESP32-S3-WROOM-1, RF_Module:ESP32-S3-WROOM-1U, symbol RF_Module:ESP32-S3-WROOM-1
- added U4: USBLC6-2SC6, Package_TO_SOT_SMD:SOT-23-6, symbol Power_Protection:USBLC6-2SC6
Connections:
- new net: D3.2 (A), J1.4 (Pin_4)
- new net: D5.2 (DOUT), D6.4 (DIN)
- new net: D4.2 (DOUT), D5.4 (DIN)
- new net +3V3: C12.1, C13.1, C14.1, C15.1, C16.1, R6.1, U3.2 (3V3)
- new net +5V: C17.1, C18.1, C19.1, C20.1, D3.1 (K), D4.1 (VDD), D5.1 (VDD), D6.1 (VDD), U4.5 (VBUS)
- new net CAN_H: J3.6 (Pin_6), J4.6 (Pin_6), J5.1 (Pin_1), J6.1 (Pin_1)
- new net CAN_L: J3.7 (Pin_7), J4.7 (Pin_7), J5.2 (Pin_2), J6.2 (Pin_2)
- new net CAN_RX: U3.9 (IO16)
- new net CAN_TX: U3.8 (IO15)
- new net ESP_EN: C10.2, C11.1, R6.2, SW1.2 (B), U3.3 (EN)
- new net GND: C10.1, C11.2, C12.2, C13.2, C14.2, C15.2, C16.2, C17.2, C18.2, C19.2, C20.2, D4.3 (VSS), D5.3 (VSS), D6.3 (VSS), J1.1 (Pin_1), J3.10 (Pin_10), J3.9 (Pin_9), J4.10 (Pin_10), J4.9 (Pin_9), J5.4 (Pin_4), J6.4 (Pin_4), SW1.1 (A), SW2.1 (A), U3.1 (GND), U3.40 (GND), U3.41 (GND), U4.2 (GND)
- new net GPIO0: SW2.2 (B), U3.27 (IO0)
- new net STATUS_LED: D4.4 (DIN), U3.11 (IO18)
- new net TSOP_OUT_1: J3.1 (Pin_1)
- new net TSOP_OUT_1_ESP: J4.1 (Pin_1), U3.12 (IO8), U3.4 (IO4)
- new net TSOP_OUT_2: J3.2 (Pin_2)
- new net TSOP_OUT_2_ESP: J4.2 (Pin_2), U3.5 (IO5)
- new net TSOP_OUT_3: J3.3 (Pin_3)
- new net TSOP_OUT_3_ESP: J4.3 (Pin_3), U3.6 (IO6)
- new net TSOP_OUT_4: J3.4 (Pin_4)
- new net TSOP_OUT_4_ESP: J4.4 (Pin_4), U3.7 (IO7)
- new net TSOP_OUT_5: J3.5 (Pin_5)
- new net TSOP_OUT_5_ESP: J4.5 (Pin_5)
- new net TX_1: U3.17 (IO9)
- new net TX_2: U3.18 (IO10)
- new net TX_3: U3.19 (IO11)
- new net TX_4: U3.20 (IO12)
- new net TX_5: U3.21 (IO13)
- new net USBC_D+: J1.2 (Pin_2), TP1.1, U4.3 (I/O2)
- new net USBC_D-: J1.3 (Pin_3), TP2.1, U4.1 (I/O1)
- new net USB_D+: TP3.1, U3.14 (USB_D+), U4.4 (I/O2)
- new net USB_D-: TP4.1, U3.13 (USB_D-), U4.6 (I/O1)
- new net VIN: J3.8 (Pin_8), J4.8 (Pin_8), J5.3 (Pin_3), J6.3 (Pin_3)
- no-connect marks 0 -> 21
Other:
- note added: "ESP32-S3"
- note added: "PROGRAMMING"
- note added: "Port IN Goes to ESP32 GPIO"
- note added: "Port OUT Goes to TSOP OUT pin"

Commit message: PTL-RAIL: IR shrouds, bottom-side node parts, test points, SW4 user button
- 3D-printed shroud outlines (28 mm) with M3 mounting holes on every LED
  and TSOP node, replicated from node 2; parts cleared from shroud areas
- TX/RX node resistors, caps and MOSFETs moved to the bottom layer and
  arranged uniformly per node
- Filleted the TSOP output bus corners; solid zone connection on the
  starved-thermal GND pads
- Silkscreen cleanup: uniform 0.8 mm refs, connector pin labels on both
  sides, J5/J6 mirrored labels, node TX/RX labels, title/company/date
- Redundant GND vias and a GND via fence along the board edge
- Mid-board mounting holes (H25-H28) and 4 mm rounded corners concentric
  with the corner holes
- Test points TP5-TP19 (TX_1-5, TSOP_OUT_1-5, VIN, +5V, +3V3, 2x GND)
  in schematic and PCB, routed
- SW4 generic user push button with R34 10k pull-up
Parts:
- added R34: 10k, Resistor_SMD:R_0805_2012Metric, symbol Device:R
- added SW4: SW_SPST, Button_Switch_SMD:SW_SPST_PTS645Sx43SMTR92, symbol Switch:SW_SPST
- added TP10: TSOP_OUT_1, TestPoint:TestPoint_Loop_D1.80mm_Drill1.0mm_Beaded, symbol Connector:TestPoint
- added TP11: TSOP_OUT_2, TestPoint:TestPoint_Loop_D1.80mm_Drill1.0mm_Beaded, symbol Connector:TestPoint
- added TP12: TSOP_OUT_3, TestPoint:TestPoint_Loop_D1.80mm_Drill1.0mm_Beaded, symbol Connector:TestPoint
- added TP13: TSOP_OUT_4, TestPoint:TestPoint_Loop_D1.80mm_Drill1.0mm_Beaded, symbol Connector:TestPoint
- added TP14: TSOP_OUT_5, TestPoint:TestPoint_Loop_D1.80mm_Drill1.0mm_Beaded, symbol Connector:TestPoint
- added TP15: VIN, TestPoint:TestPoint_Loop_D1.80mm_Drill1.0mm_Beaded, symbol Connector:TestPoint
- added TP16: +5V, TestPoint:TestPoint_Loop_D1.80mm_Drill1.0mm_Beaded, symbol Connector:TestPoint
- added TP17: +3V3, TestPoint:TestPoint_Loop_D1.80mm_Drill1.0mm_Beaded, symbol Connector:TestPoint
- added TP18, TP19: GND, TestPoint:TestPoint_Loop_D1.80mm_Drill1.0mm_Beaded, symbol Connector:TestPoint
- added TP5: TX_1, TestPoint:TestPoint_Loop_D1.80mm_Drill1.0mm_Beaded, symbol Connector:TestPoint
- added TP6: TX_2, TestPoint:TestPoint_Loop_D1.80mm_Drill1.0mm_Beaded, symbol Connector:TestPoint
- added TP7: TX_3, TestPoint:TestPoint_Loop_D1.80mm_Drill1.0mm_Beaded, symbol Connector:TestPoint
- added TP8: TX_4, TestPoint:TestPoint_Loop_D1.80mm_Drill1.0mm_Beaded, symbol Connector:TestPoint
- added TP9: TX_5, TestPoint:TestPoint_Loop_D1.80mm_Drill1.0mm_Beaded, symbol Connector:TestPoint
- U3: footprint RF_Module:ESP32-S3-WROOM-1U -> RF_Module:ESP32-S3-WROOM-1
Connections:
- net +3V3: now also R34.1, TP17.1
- net +5V: now also TP16.1
- net CAN_H: now also J4.5 (Pin_5), J6.4 (Pin_4); no longer J4.6 (Pin_6), J6.1 (Pin_1)
- net CAN_L: now also J4.4 (Pin_4), J6.3 (Pin_3); no longer J4.7 (Pin_7), J6.2 (Pin_2)
- net GND: now also J4.1 (Pin_1), J4.2 (Pin_2), J6.1 (Pin_1), SW4.2 (B), TP18.1, TP19.1; no longer J4.10 (Pin_10), J4.9 (Pin_9), J6.4 (Pin_4)
- net TSOP_OUT_1: now also TP10.1
- net TSOP_OUT_1_ESP: now also J4.10 (Pin_10); no longer J4.1 (Pin_1), U3.12 (IO8)
- net TSOP_OUT_2: now also TP11.1
- net TSOP_OUT_2_ESP: now also J4.9 (Pin_9); no longer J4.2 (Pin_2)
- net TSOP_OUT_3: now also TP12.1
- net TSOP_OUT_3_ESP: now also J4.8 (Pin_8); no longer J4.3 (Pin_3)
- net TSOP_OUT_4: now also TP13.1
- net TSOP_OUT_4_ESP: now also J4.7 (Pin_7); no longer J4.4 (Pin_4)
- net TSOP_OUT_5: now also TP14.1
- net TSOP_OUT_5_ESP: now also J4.6 (Pin_6), U3.12 (IO8); no longer J4.5 (Pin_5)
- net TX_1: now also TP5.1
- net TX_2: now also TP6.1
- net TX_3: now also TP7.1
- net TX_4: now also TP8.1
- net TX_5: now also TP9.1
- net VIN: now also J4.3 (Pin_3), J6.2 (Pin_2), TP15.1; no longer J4.8 (Pin_8), J6.3 (Pin_3)
- net at U3.26 (IO45): now also R34.2, SW4.1 (A)
- no-connect marks 21 -> 20

Commit message: PTL-RAIL: move SW4 user button to IO14 (ACK_BUTTON), add C27 100nF debounce
Parts:
- added C27: 0.1uF, Capacitor_SMD:C_0805_2012Metric, symbol Device:C
Connections:
- net GND: now also C27.2
- net ACK_BUTTON: now reaches R34.2, SW4.1 (A)
- net ACK_BUTTON: now also U3.22 (IO14), C27.1; no longer U3.26 (IO45)
- no-connect marks 20 -> 19
Changed lines of the file:
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@@
 	)
 	(junction
+		(at 111.76 135.89)
+		(diameter 0)
+		(color 0 0 0 0)
+	)
+	(junction
 		(at 185.42 92.71)
 		(diameter 0)
@@
 	)
 	(junction
-		(at 111.76 135.89)
+		(at 35.56 97.79)
 		(diameter 0)
 		(color 0 0 0 0)
 	)
 	(junction
-		(at 35.56 97.79)
+		(at 20.32 118.11)
 		(diameter 0)
 		(color 0 0 0 0)
 	)
 	(junction
-		(at 20.32 118.11)
+		(at 350.52 88.9)
 		(diameter 0)
 		(color 0 0 0 0)
 	)
 	(junction
-		(at 350.52 88.9)
+		(at 127 140.97)
 		(diameter 0)
 		(color 0 0 0 0)
@@
 	)
 	(no_connect
-		(at 69.85 138.43)
-	)
-	(no_connect
 		(at 69.85 107.95)
 	)
@@
 	(wire
 		(pts
+			(xy 69.85 138.43) (xy 44.45 138.43)
+		)
+		(stroke
+			(width 0)
+			(type default)
+		)
+	)
+	(wire
+		(pts
 			(xy 172.72 90.17) (xy 173.99 90.17)
 		)
@@
 	(wire
 		(pts
+			(xy 109.22 135.89) (xy 111.76 135.89)
+		)
+		(stroke
+			(width 0)
+			(type default)
+		)
+	)
+	(wire
+		(pts
 			(xy 185.42 92.71) (xy 194.31 92.71)
 		)
@@
 	(wire
 		(pts
+			(xy 127 140.97) (xy 127 135.89)
+		)
+		(stroke
+			(width 0)
+			(type default)
+		)
+	)
+	(wire
+		(pts
 			(xy 322.58 88.9) (xy 330.2 88.9)
 		)
@@
 	(wire
 		(pts
+			(xy 123.19 140.97) (xy 127 140.97)
+		)
+		(stroke
+			(width 0)
+			(type default)
+		)
+	)
+	(wire
+		(pts
 			(xy 69.85 135.89) (xy 44.45 135.89)
 		)
@@
 	(wire
 		(pts
+			(xy 111.76 140.97) (xy 115.57 140.97)
+		)
+		(stroke
+			(width 0)
+			(type default)
+		)
+	)
+	(wire
+		(pts
 			(xy 182.88 100.33) (xy 182.88 99.06)
 		)
@@
 		)
 	)
-	(bus
+	(wire
 		(pts
-			(xy 227.33 69.85) (xy 224.79 67.31)
+			(xy 127 144.78) (xy 127 140.97)
 		)
 		(stroke
@@
 		)
 	)
-	(wire
+	(bus
 		(pts
-			(xy 128.27 135.89) (xy 124.46 135.89)
+			(xy 227.33 69.85) (xy 224.79 67.31)
 		)
 		(stroke
@@
 	(wire
 		(pts
+			(xy 111.76 135.89) (xy 111.76 140.97)
+		)
+		(stroke
+			(width 0)
+			(type default)
+		)
+	)
+	(wire
+		(pts
 			(xy 355.6 83.82) (xy 358.14 83.82)
 		)
@@
 	(wire
 		(pts
+			(xy 127 135.89) (xy 124.46 135.89)
+		)
+		(stroke
+			(width 0)
+			(type default)
+		)
+	)
+	(wire
+		(pts
 			(xy 392.43 71.12) (xy 377.19 71.12)
 		)
@@
 	(wire
 		(pts
-			(xy 100.33 135.89) (xy 111.76 135.89)
-		)
-		(stroke
-			(width 0)
-			(type default)
-		)
-	)
-	(wire
-		(pts
 			(xy 160.02 90.17) (xy 172.72 90.17)
 		)
@@
 		)
 	)
+	(label "ACK_BUTTON"
+		(at 109.22 135.89 270)
+		(effects
+			(font
+				(size 1.27 1.27)
+			)
+			(justify right bottom)
+		)
+	)
 	(label "TX_2"
 		(at 213.36 83.82 0)
@@
 		)
 	)
+	(label "ACK_BUTTON"
+		(at 44.45 138.43 0)
+		(effects
+			(font
+				(size 1.27 1.27)
+			)
+			(justify left bottom)
+		)
+	)
 	(label "USB_D-"
 		(at 194.31 90.17 0)
@@
 	(symbol
 		(lib_id "power:GND")
-		(at 128.27 135.89 0)
+		(at 127 144.78 0)
 		(unit 1)
 		(body_style 1)
@@
 		(fields_autoplaced yes)
 		(property "Reference" "#PWR066"
-			(at 128.27 142.24 0)
+			(at 127 151.13 0)
 			(hide yes)
 			(show_name no)
@@
 		)
 		(property "Value" "GND"
-			(at 128.27 140.97 0)
+			(at 127 149.86 0)
 			(show_name no)
 			(do_not_autoplace no)
@@
 		)
 		(property "Footprint" ""
-			(at 128.27 135.89 0)
+			(at 127 144.78 0)
 			(hide yes)
 			(show_name no)
@@
 		)
 		(property "Datasheet" ""
-			(at 128.27 135.89 0)
+			(at 127 144.78 0)
 			(hide yes)
 			(show_name no)
@@
 		)
 		(property "Description" "Power symbol creates a global label with name \"GND\" , ground"
-			(at 128.27 135.89 0)
+			(at 127 144.78 0)
 			(hide yes)
 			(show_name no)
@@
 					(unit 1)
 				)
+			)
+		)
+	)
+	(symbol
+		(lib_id "Device:C")
+		(at 119.38 140.97 90)
+		(unit 1)
+		(body_style 1)
+		(exclude_from_sim no)
+		(in_bom yes)
+		(on_board yes)
+		(in_pos_files yes)
+		(dnp no)
+		(property "Reference" "C27"
+			(at 116.84 139.7 90)
+			(show_name no)
+			(do_not_autoplace no)
+			(effects
+				(font
+					(size 0.8 0.8)
+				)
+				(justify left)
+			)
+		)
+		(property "Value" "0.1uF"
+			(at 123.19 144.78 90)
+			(show_name no)
+			(do_not_autoplace no)
+			(effects
+				(font
+					(size 0.8 0.8)
+				)
+				(justify left)
+			)
+		)
+		(property "Footprint" "Capacitor_SMD:C_0805_2012Metric"
+			(at 123.19 140.0048 0)
+			(hide yes)
+			(show_name no)
+			(do_not_autoplace no)
+			(effects
+				(font
+					(size 1.27 1.27)
+				)
+			)
+		)
+		(property "Datasheet" ""
+			(at 119.38 140.97 0)
+			(hide yes)
+			(show_name no)
+			(do_not_autoplace no)
+			(effects
+				(font
+					(size 1.27 1.27)
+				)
+			)
+		)
+		(property "Description" "Unpolarized capacitor"
+			(at 119.38 140.97 0)
+			(hide yes)
+			(show_name no)
+			(do_not_autoplace no)
+			(effects
+				(font
+					(size 1.27 1.27)
+				)
+			)
+		)
+		(pin "1"
+		)
+		(pin "2"
+		)
+		(instances
+			(project "PTL-RAIL"
+				(path "/f069ed8f-812c-4c88-b7da-e87f505ec63b/843560ab-5821-40bc-86d9-e72d8423fdb4"
+					(reference "C27")
+					(unit 1)
+				)

Commit message: PTL-RAIL rev A: normalize cap values, IO45 no-connect, README and docs
- Capacitor values unified: 0.1uF -> 100nF (C10, C16-C21, C27; now one
  BOM line with C5), '4.7 µF' -> 4.7uF (C22-C26)
- No-connect flag on U3 IO45 (ERC clean apart from 2 CAN label warnings)
- Zones refilled
- PTL-RAIL/README.md: board summary, pinouts, ESP32 pin map, test points,
  mounting, fab/assembly notes, production file list, rev A open issues
- Root README points to PTL-RAIL and the release assets
Parts:
- C10, C16, C17, C18, C19, C20, C27: value 0.1uF -> 100nF
Connections:
- no-connect marks 19 -> 20
Changed lines of the file:
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@@
 	)
 	(no_connect
+		(at 100.33 135.89)
+	)
+	(no_connect
 		(at 100.33 118.11)
 	)
@@
 			)
 		)
-		(property "Value" "0.1uF"
+		(property "Value" "100nF"
 			(at 250.19 118.11 0)
 			(show_name no)
@@
 			)
 		)
-		(property "Value" "0.1uF"
+		(property "Value" "100nF"
 			(at 123.19 144.78 90)
 			(show_name no)
@@
 			)
 		)
-		(property "Value" "0.1uF"
+		(property "Value" "100nF"
 			(at 271.78 118.11 0)
 			(show_name no)
@@
 			)
 		)
-		(property "Value" "0.1uF"
+		(property "Value" "100nF"
 			(at 180.34 119.38 0)
 			(show_name no)
@@
 			)
 		)
-		(property "Value" "0.1uF"
+		(property "Value" "100nF"
 			(at 228.6 118.11 0)
 			(show_name no)
@@
 			)
 		)
-		(property "Value" "0.1uF"
+		(property "Value" "100nF"
 			(at 125.73 64.7699 0)
 			(show_name no)
@@
 			)
 		)
-		(property "Value" "0.1uF"
+		(property "Value" "100nF"
 			(at 33.02 106.68 90)
 			(show_name no)
